Commit message: Handshake controller stub; Added franka_description submodule

File: franka_handshake_description/robots/common/franka_arm.ros2_control.xacro (robot description, xacro)
@@ -89,5 +89,5 @@
       <gazebo>
         <plugin filename="franka_ign_ros2_control-system" name="ign_ros2_control::IgnitionROS2ControlPlugin">
-          <parameters>$(find franka_gazebo_bringup)/config/franka_gazebo_controllers.yaml</parameters>
+          <parameters>$(find franka_handshake_gazebo_bringup)/config/franka_handshake_gazebo_controllers.yaml</parameters>
         </plugin>
       </gazebo>

File: franka_handshake_description/robots/common/franka_robot.xacro (robot description, xacro)
@@ -140,5 +140,5 @@
     </xacro:if>
     <xacro:if value="${ros2_control}">
-      <xacro:include filename="$(find franka_description)/robots/common/franka_arm.ros2_control.xacro"/>
+      <xacro:include filename="$(find franka_handshake_description)/robots/common/franka_arm.ros2_control.xacro"/>
       <xacro:franka_arm_ros2_control
           arm_id="${arm_id}"

File: franka_handshake_description/urdf/franka_handshake.urdf.xacro (robot description, xacro)
@@ -10,13 +10,15 @@
   <xacro:include filename="$(find franka_handshake_description)/urdf/franka_handshake/franka_handshake_macro.xacro"/>
   <xacro:include filename="$(find franka_handshake_description)/urdf/franka_handshake/franka_handshake_macro.ros2_control.xacro"/>
-  <xacro:include filename="$(find franka_description)/robots/common/franka_robot.xacro"/>
+  <xacro:include filename="$(find franka_handshake_description)/robots/common/franka_robot.xacro"/>
   <xacro:include filename="$(find mekahand_description)/urdf/mekahand/mekahand_macro.xacro"/>
   <!-- create link fixed to the "world" -->
-  <link name="world"/>
-  <joint name="world_to_base" type="fixed">
-    <parent link="world"/>
-    <child link="base"/> <!-- or whatever the root link of franka_robot is -->
-    <origin xyz="0 0 0" rpy="0 0 0"/>
-  </joint>
+  <xacro:if value="false">
+    <link name="my_base"/>
+    <joint name="my_base_to_base" type="fixed">
+      <parent link="my_base"/>
+      <child link="base"/> <!-- or whatever the root link of franka_robot is -->
+      <origin xyz="0 0 0" rpy="0 0 0"/>
+    </joint>
+  </xacro:if>
   <xacro:arg name="arm_id" default="fr3" />
   <!-- The prefix of the robot -->
